File: Eval-GP-Board/General Purpose Op Amp Eval-Board.kicad_pcb (KiCad board)
At the start: 2 copper layers, 68 parts, among them J2 Conn_01x03_Male, U1 ADA4522-2, U2 ADA4075-2, U3 ADA4807-2ARM

Commit message: update-version
Other:
- board outline added: 81.3 x 53.3 mm
Changed lines of the file:
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@@
   (general
     (thickness 1.6)
-    (drawings 4)
+    (drawings 8)
     (tracks 298)
     (zones 0)
@@
     )
   )
+  (gr_line (start 127 52.07) (end 45.72 52.07) (layer Edge.Cuts) (width 0.05))
+  (gr_line (start 127 105.41) (end 127 52.07) (layer Edge.Cuts) (width 0.05))
+  (gr_line (start 45.72 105.41) (end 127 105.41) (layer Edge.Cuts) (width 0.05))
+  (gr_line (start 45.72 52.07) (end 45.72 105.41) (layer Edge.Cuts) (width 0.05))
   (gr_line (start 127 52.07) (end 45.72 52.07) (layer F.SilkS) (width 0.12))
   (gr_line (start 127 105.41) (end 127 52.07) (layer F.SilkS) (width 0.12))
