File: eval-board-ADA4817-1/eval-board-ADA4817-1.sch (KiCad schematic (older format))
At the start: 27 parts, among them J2 -VIN, J3 +VIN, J4 Conn_01x03_Male, J5 VOUT, U1 ADA4817-1

Commit message: updated
Parts:
- added JP1: Jumper_3_Open, Jumper:SolderJumper-3_P1.3mm_Open_RoundedPad1.0x1.5mm_NumberLabels, symbol Jumper:Jumper_3_Open
- added RF2, RF3: R, Resistor_SMD:R_0603_1608Metric_Pad1.05x0.95mm_HandSolder, symbol Device:R
- added RV1: R_POT, Connector_PinSocket_2.54mm:PinSocket_1x03_P2.54mm_Vertical, symbol Device:R_POT
- C1, C2, C6, C7, C8, C9: footprint Capacitor_SMD:C_0603_1608Metric -> Capacitor_SMD:C_0603_1608Metric_Pad1.05x0.95mm_HandSolder
- C10, C4: footprint Capacitor_SMD:CP_Elec_4x5.3 -> Capacitor_SMD:CP_Elec_4x5.4
- CF: renamed from C3; value CF -> C; footprint Capacitor_SMD:C_0603_1608Metric -> Capacitor_SMD:C_0603_1608Metric_Pad1.05x0.95mm_HandSolder
- CL: renamed from C5; value CL -> C; footprint Capacitor_SMD:C_0603_1608Metric -> Capacitor_SMD:C_0603_1608Metric_Pad1.05x0.95mm_HandSolder
- J4: footprint Connector_PinSocket_2.54mm:PinSocket_1x03_P2.54mm_Vertical -> Connector_JST:JST_XH_B3B-XH-A_1x03_P2.50mm_Vertical
- R1, R10, R11, R12, R4, R5, R6, R7: footprint Resistor_SMD:R_0603_1608Metric -> Resistor_SMD:R_0603_1608Metric_Pad1.05x0.95mm_HandSolder
- RF1: renamed from R8; value RF -> R; footprint Resistor_SMD:R_0603_1608Metric -> Resistor_SMD:R_0603_1608Metric_Pad1.05x0.95mm_HandSolder
- RS: renamed from R9; value RS -> R; footprint Resistor_SMD:R_0603_1608Metric -> Resistor_SMD:R_0603_1608Metric_Pad1.05x0.95mm_HandSolder
- RTN: renamed from R2; value RTN -> R; footprint Resistor_SMD:R_0603_1608Metric -> Resistor_SMD:R_0603_1608Metric_Pad1.05x0.95mm_HandSolder
- RTP: renamed from R3; value RTP -> R; footprint Resistor_SMD:R_0603_1608Metric -> Resistor_SMD:R_0603_1608Metric_Pad1.05x0.95mm_HandSolder
Connections:
- net GNDREF: now also C10.1; no longer C10.2
- net VEE: now also C10.2; no longer C10.1
- net at CF.1, U1.1 (FB): now also JP1.2 (C); no longer RF1.1
- net at CF.2, R5.1, R6.2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: now also RF1.1, RF2.1, RF3.2, RV1.1; no longer RF1.2
- new net: JP1.1 (A), RF1.2, RF2.2, RF3.1
- new net: JP1.3 (B), RV1.2
Other:
- moved on the sheet: C1, C10, C2, C4, C6, C7, C8, C9, CF, CL, J2, J3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
